File: Hardware/MeshThing.sch (KiCad schematic (older format))
At the start: 25 parts, among them IC1 ATMEGA2564/1284/644RFR2, SW1 RST, U1 CONN_MICROSD, U2 XBEE

Commit message: Begin v1.2. Cleanup done.
Parts:
- R2, R3: value 330 -> 270
Changed lines of the file:
@@
 P 2650 1050
 F 0 "R2" V 2730 1050 40  0000 C CNN
-F 1 "330" V 2657 1051 40  0000 C CNN
+F 1 "270" V 2657 1051 40  0000 C CNN
 F 2 "" V 2580 1050 30  0000 C CNN
 F 3 "" H 2650 1050 30  0000 C CNN
@@
 P 4300 1050
 F 0 "R3" V 4380 1050 40  0000 C CNN
-F 1 "330" V 4307 1051 40  0000 C CNN
+F 1 "270" V 4307 1051 40  0000 C CNN
 F 2 "" V 4230 1050 30  0000 C CNN
 F 3 "" H 4300 1050 30  0000 C CNN
