File: Hardware/MeshThing.sch (KiCad schematic (older format))
At the start: 25 parts, among them IC1 ATMEGA2564/1284/644RFR2, SW1 RST, U1 CONN_MICROSD, U2 XBEE

Commit message: Initial v2.0 commit.
Parts:
- removed A1: Antenna, symbol CONN_4
- removed C9: 100n, symbol C
- removed D1, D2: LED, symbol LED
- removed H2: ICSP, symbol CONN_3X2
- removed R2, R3: 270, symbol R
- removed SJ1, SJ2: SMTJPR, symbol BREAKER
- removed SW1: RST, symbol SPST
- removed U1: CONN_MICROSD, symbol CONN_MICROSD
- removed U2: XBEE, symbol XBEE
- removed XTAL1: 16MHz, CSM-3X, symbol CRYSTAL
- added A1: ANTENNA, symbol CONN_2
- added F1, F2, F3: CONN_1, symbol CONN_1
- added H1: ICSP, symbol CONN_3X2
- added P1: CONN34, symbol CONN34
- added S1: RFShield, symbol CONN_1
- added XTAL1: CRYSTAL_SMD-TSX3225, symbol CRYSTAL_SMD-TSX3225
- C3, C4: value 39p -> 10p
Connections:
- net labels added: PB6, PB7, PD4, PD5, PD6, PD7, PE2, PE3, PE7, PG1
- wire segments 168 -> 148
- no-connect marks 16 -> 4
Other:
- note added: "Fiducials"
- note added: "Footprint Pins"
- note removed: "Activity LED?"
- note removed: "Buffers Needed? Don't think so.\nAlready at 3.3v, no V-divider."
- note removed: "Changing R3 to be <10k as the green LEDs currently on BOM from v1.0 are dim. \n\nNeed to consult the datasheet further for current profile."
- note removed: "D1/D2 are optimal at 10-20mA with drop of 2.1-2.2V. Changing R2/R3 to be 330\neven though that doesn't calculate out right, but being concervative in case 5v\ncomes across them. Need to update BOM for v1.1."
- note removed: "Needed:\nPower LED - Done.\nOther Indicators?"

Commit message: Very nearly there.
Parts:
- added C9: 100n, symbol C
Connections:
- net +3.3V: now also C9.1
- net GND: now also C9.2
Changed lines of the file:
@@
 Connection ~ 6100 2050
 Wire Wire Line
-	7200 1500 6100 1500
+	5350 1500 7200 1500
 Connection ~ 7200 1500
 Connection ~ 4700 2600
@@
 Wire Wire Line
 	9350 2100 9050 2100
+$Comp
+L C C9
+U 1 1 52B8322D
+P 5350 1700
+F 0 "C9" H 5350 1800 40  0000 L CNN
+F 1 "100n" H 5356 1615 40  0000 L CNN
+F 2 "" H 5388 1550 30  0000 C CNN
+F 3 "" H 5350 1700 60  0000 C CNN
+	1    5350 1700
+	1    0    0    -1
+$EndComp
+Connection ~ 6100 1500
+$Comp
+L GND #PWR011
+U 1 1 52B83301
+P 5350 2000
+F 0 "#PWR011" H 5350 2000 30  0001 C CNN
+F 1 "GND" H 5350 1930 30  0001 C CNN
+F 2 "" H 5350 2000 60  0000 C CNN
+F 3 "" H 5350 2000 60  0000 C CNN
+	1    5350 2000
+	1    0    0    -1
+$EndComp
+Wire Wire Line
+	5350 1900 5350 2000
 $EndSCHEMATC

Commit message: Removed ICSP pads.
Parts:
- removed H1: ICSP, symbol CONN_3X2
Changed lines of the file:
@@
 	3600 6800 3500 6800
-Wire Wire Line
-	9050 1950 9350 1950
-Wire Wire Line
-	10150 1950 10250 1950
 Wire Wire Line
 	9150 1800 9050 1800
@@
 Footprint Pins
 $Comp
-L CONN_3X2 H1
-U 1 1 52B66679
-P 9750 2000
-F 0 "H1" H 9750 2250 50  0000 C CNN
-F 1 "ICSP" V 9750 2050 40  0000 C CNN
-F 2 "" H 9750 2000 60  0000 C CNN
-F 3 "" H 9750 2000 60  0000 C CNN
-	1    9750 2000
-	1    0    0    -1
-$EndComp
-Text GLabel 9050 2100 0    60   Input ~ 0
-Reset
-$Comp
-L GND #PWR09
-U 1 1 52B666D4
-P 10300 2200
-F 0 "#PWR09" H 10300 2200 30  0001 C CNN
-F 1 "GND" H 10300 2130 30  0001 C CNN
-F 2 "" H 10300 2200 60  0000 C CNN
-F 3 "" H 10300 2200 60  0000 C CNN
-	1    10300 2200
-	1    0    0    -1
-$EndComp
-$Comp
-L +3.3V #PWR010
-U 1 1 52B666DF
-P 10300 1750
-F 0 "#PWR010" H 10300 1710 30  0001 C CNN
-F 1 "+3.3V" H 10300 1860 30  0000 C CNN
-F 2 "" H 10300 1750 60  0000 C CNN
-F 3 "" H 10300 1750 60  0000 C CNN
-	1    10300 1750
-	1    0    0    -1
-$EndComp
-Wire Wire Line
-	10150 2050 10300 2050
-Wire Wire Line
-	10300 2050 10300 2200
-Wire Wire Line
-	10150 1850 10300 1850
-Wire Wire Line
-	10300 1850 10300 1750
-Wire Wire Line
-	9350 1850 9150 1850
-Connection ~ 9150 1850
-Wire Wire Line
-	9350 2050 9350 2100
-Wire Wire Line
-	9350 2100 9050 2100
-$Comp
 L C C9
 U 1 1 52B8322D
@@
 Wire Wire Line
 	5350 1900 5350 2000
+Wire Wire Line
+	9250 1950 9050 1950
+Wire Wire Line
+	10200 1950 10250 1950
 $EndSCHEMATC
