File: Hardware/MeshThing.kicad_pcb (KiCad board)
At the start: 4 copper layers, 19.1 x 24.7 mm, 22 parts, among them IC1 ATMEGA2564/1284/644RFR2, P1 CONN34

Commit message: Very nearly there.
Parts:
- added C9: 100n, SMD_Packages:SM0402_c, F.Cu at (151.4, 96.1)
Routing:
- net +3.3V: track 59.2 -> 61.1 mm
- net GND: track 94.8 -> 96.3 mm

Commit message: Logo work.
Parts:
- added VAL: M9Logo-scaled, _MT_M9Logo-Scaled:M9Logo-scaled, F.Cu at (143.0, 90.5)
- PrettyLady: moved to B.Cu
- moved PrettyLady 18.1 mm to (150.3, 106.9)
- moved G*** 0.05 mm to (157.0, 90.5)
Changed lines of the file:
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@@
     (links 85)
     (no_connects 0)
-    (area 140.349999 87.569999 159.650001 112.430001)
+    (area 136.629829 85.2768 169.635341 113.0282)
     (thickness 1.6)
     (drawings 7)
     (tracks 588)
     (zones 0)
-    (modules 23)
+    (modules 24)
     (nets 47)
   )
@@
   (layers
     (15 F.Cu signal)
-    (2 Inner2.Cu power)
-    (1 Inner1.Cu signal)
-    (0 B.Cu signal)
+    (2 Inner2.Cu power hide)
+    (1 Inner1.Cu signal hide)
+    (0 B.Cu signal hide)
     (16 B.Adhes user hide)
     (17 F.Adhes user hide)
@@
       (clearance 0.375))
   )
-  (module _MT_MC_Pretty:_MC_LOGO-PrettyLady (layer F.Cu)
-    (at 142.9 90.32)
-    (fp_text reference PrettyLady (at 0 3.302) (layer F.SilkS) hide
-      (effects (font (thickness 0.3048)))
-    )
-    (fp_text value PrettyLady (at 0 -3.302) (layer F.SilkS) hide
-      (effects (font (thickness 0.3048)))
+  (module _MT_MC_Pretty:_MC_LOGO-PrettyLady (layer B.Cu)
+    (at 150.27 106.86)
+    (fp_text reference PrettyLady (at 0 -3.302) (layer B.SilkS) hide
+      (effects (font (thickness 0.3048)) (justify mirror))
+    )
+    (fp_text value PrettyLady (at 0 3.302) (layer B.SilkS) hide
+      (effects (font (thickness 0.3048)) (justify mirror))
     )
     (fp_poly (pts (xy 2.413 -2.5019) (xy 0.10668 -2.47904) (xy -2.19964 -2.45364) (xy -2.22504 0.0635)
       (xy -2.2479 2.58064) (xy -2.26822 0.02032) (xy -2.286 -2.54) (xy 0.0635 -2.52222)
-      (xy 2.413 -2.5019) (xy 2.413 -2.5019)) (layer F.SilkS) (width 0.00254))
+      (xy 2.413 -2.5019) (xy 2.413 -2.5019)) (layer B.SilkS) (width 0.00254))
     (fp_poly (pts (xy 0.59182 2.45364) (xy 0.51054 2.4892) (xy 0.27432 2.51714) (xy -0.09652 2.53238)
       (xy -0.58166 2.54) (xy -1.0541 2.53746) (xy -1.38684 2.5273) (xy -1.61036 2.50952)
@@
       (xy -0.34036 1.72212) (xy -0.27432 1.82626) (xy -0.1143 1.97104) (xy -0.04318 2.0193)
       (xy 0.1397 2.16154) (xy 0.24384 2.27076) (xy 0.254 2.29616) (xy 0.32258 2.35458)
-      (xy 0.42164 2.36982) (xy 0.5588 2.40538) (xy 0.59182 2.45364) (xy 0.59182 2.45364)) (layer F.SilkS) (width 0.00254))
+      (xy 0.42164 2.36982) (xy 0.5588 2.40538) (xy 0.59182 2.45364) (xy 0.59182 2.45364)) (layer B.SilkS) (width 0.00254))
     (fp_poly (pts (xy 1.75768 0.42418) (xy 1.73228 0.82042) (xy 1.6891 1.07188) (xy 1.6891 -0.04826)
       (xy 1.6891 -0.19304) (xy 1.62814 -0.254) (xy 1.4986 -0.21082) (xy 1.31572 -0.1016)
@@
       (xy 0.84582 -0.89662) (xy 0.90424 -0.90678) (xy 1.18872 -0.94996) (xy 1.36398 -0.94742)
       (xy 1.4859 -0.89408) (xy 1.55448 -0.83566) (xy 1.651 -0.65786) (xy 1.7145 -0.36068)
-      (xy 1.7526 0.01524) (xy 1.75768 0.42418) (xy 1.75768 0.42418)) (layer F.SilkS) (width 0.00254))
+      (xy 1.7526 0.01524) (xy 1.75768 0.42418) (xy 1.75768 0.42418)) (layer B.SilkS) (width 0.00254))
     (fp_poly (pts (xy 1.84658 1.47574) (xy 1.83134 1.54432) (xy 1.8034 1.5494) (xy 1.79324 1.41478)
       (xy 1.79324 1.397) (xy 1.80594 1.26492) (xy 1.83134 1.27762) (xy 1.83642 1.29032)
-      (xy 1.84658 1.47574) (xy 1.84658 1.47574)) (layer F.SilkS) (width 0.00254))
+      (xy 1.84658 1.47574) (xy 1.84658 1.47574)) (layer B.SilkS) (width 0.00254))
     (fp_poly (pts (xy -1.37668 -0.09398) (xy -1.37922 0.14986) (xy -1.397 0.3175) (xy -1.4478 0.67564)
       (xy -1.50368 0.88138) (xy -1.57988 0.94742) (xy -1.68402 0.89408) (xy -1.7526 0.8255)
@@
       (xy -2.01676 -0.36322) (xy -1.94564 -0.54864) (xy -1.93548 -0.65786) (xy -1.9177 -0.75946)
       (xy -1.82118 -0.7493) (xy -1.68148 -0.64262) (xy -1.5367 -0.4699) (xy -1.42494 -0.27686)
-      (xy -1.37668 -0.09398) (xy -1.37668 -0.09398)) (layer F.SilkS) (width 0.00254))
+      (xy -1.37668 -0.09398) (xy -1.37668 -0.09398)) (layer B.SilkS) (width 0.00254))
     (fp_poly (pts (xy -0.84836 0.46482) (xy -0.889 0.508) (xy -0.93218 0.46482) (xy -0.889 0.42164)
-      (xy -0.84836 0.46482) (xy -0.84836 0.46482)) (layer F.SilkS) (width 0.00254))
+      (xy -0.84836 0.46482) (xy -0.84836 0.46482)) (layer B.SilkS) (width 0.00254))
     (fp_poly (pts (xy 0.67564 0.889) (xy 0.635 0.92964) (xy 0.59182 0.889) (xy 0.635 0.84582)
-      (xy 0.67564 0.889) (xy 0.67564 0.889)) (layer F.SilkS) (width 0.00254))
+      (xy 0.67564 0.889) (xy 0.67564 0.889)) (layer B.SilkS) (width 0.00254))
     (fp_poly (pts (xy 1.57988 -0.05842) (xy 1.56718 -0.00762) (xy 1.524 0) (xy 1.45288 -0.03302)
-      (xy 1.46558 -0.05842) (xy 1.56718 -0.06858) (xy 1.57988 -0.05842) (xy 1.57988 -0.05842)) (layer F.SilkS) (width 0.00254))
+      (xy 1.46558 -0.05842) (xy 1.56718 -0.06858) (xy 1.57988 -0.05842) (xy 1.57988 -0.05842)) (layer B.SilkS) (width 0.00254))
   )
   (module _MT_MC_Pretty:_MC_pin_pad_3x2 (layer B.Cu)
@@
   )
   (module _MT_OHW_LOGO:LOGO (layer F.Cu)
-    (at 157.05 90.55)
+    (at 157 90.55)
     (fp_text reference G*** (at 0 2.38506) (layer F.SilkS) hide
       (effects (font (size 0.2032 0.2032) (thickness 0.04064)))
@@
       (net 2 GND))
   )
+  (module _MT_M9Logo-Scaled:M9Logo-scaled (layer F.Cu)
+    (at 143 90.55)
+    (fp_text reference VAL (at 0 0) (layer F.SilkS) hide
+      (effects (font (size 1.143 1.143) (thickness 0.1778)))
+    )
+    (fp_text value M9Logo-scaled (at 0 0) (layer F.SilkS) hide
+      (effects (font (size 1.143 1.143) (thickness 0.1778)))
+    )
+    (fp_poly (pts (xy 2.05486 -0.40132) (xy 2.05232 -0.37084) (xy 2.04216 -0.29464) (xy 2.02692 -0.18542)
+      (xy 2.00406 -0.04318) (xy 1.97866 0.12192) (xy 1.94818 0.3048) (xy 1.94056 0.35052)
+      (xy 1.8161 1.07442) (xy 1.2573 1.55194) (xy 1.1684 1.62814) (xy 1.1684 0.08636)
+      (xy 1.1684 0.0127) (xy 1.1684 -0.2159) (xy 1.16586 -0.39878) (xy 1.16078 -0.54102)
+      (xy 1.15316 -0.65278) (xy 1.14046 -0.7366) (xy 1.12014 -0.79756) (xy 1.09474 -0.84582)
+      (xy 1.05918 -0.88392) (xy 1.016 -0.91948) (xy 0.9906 -0.93472) (xy 0.93726 -0.9652)
+      (xy 0.88646 -0.98298) (xy 0.81534 -0.98806) (xy 0.71374 -0.98806) (xy 0.70358 -0.98552)
+      (xy 0.59944 -0.98044) (xy 0.53594 -0.97028) (xy 0.49022 -0.94996) (xy 0.44958 -0.91694)
+      (xy 0.4191 -0.88646) (xy 0.36068 -0.80518) (xy 0.32004 -0.70358) (xy 0.29464 -0.57404)
+      (xy 0.28194 -0.40894) (xy 0.2794 -0.28448) (xy 0.28702 -0.10668) (xy 0.31496 0.03048)
+      (xy 0.36068 0.12954) (xy 0.42672 0.19812) (xy 0.45974 0.21844) (xy 0.55372 0.24384)
+      (xy 0.6604 0.24638) (xy 0.75692 0.22352) (xy 0.8128 0.1905) (xy 0.83566 0.17018)
+      (xy 0.8509 0.17018) (xy 0.85852 0.19304) (xy 0.8636 0.25146) (xy 0.8636 0.34798)
+      (xy 0.8636 0.3937) (xy 0.85852 0.53594) (xy 0.84582 0.635) (xy 0.81788 0.6985)
+      (xy 0.7747 0.72898) (xy 0.72136 0.7366) (xy 0.6604 0.71374) (xy 0.6223 0.65024)
+      (xy 0.6096 0.54864) (xy 0.6096 0.4572) (xy 0.4699 0.4572) (xy 0.3302 0.4572)
+      (xy 0.3302 0.59944) (xy 0.34544 0.73914) (xy 0.39116 0.8509) (xy 0.46228 0.93218)
+      (xy 0.55372 0.98806) (xy 0.6731 1.016) (xy 0.8001 1.01854) (xy 0.92202 0.99314)
+      (xy 1.01092 0.94742) (xy 1.0541 0.9144) (xy 1.08966 0.87884) (xy 1.11506 0.83566)
+      (xy 1.13538 0.77978) (xy 1.15062 0.70358) (xy 1.15824 0.60198) (xy 1.16332 0.4699)
+      (xy 1.1684 0.29972) (xy 1.1684 0.08636) (xy 1.1684 1.62814) (xy 0.6985 2.02946)
+      (xy 0.1016 2.02946) (xy 0.1016 0.9906) (xy 0.1016 0) (xy 0.1016 -0.9906)
+      (xy -0.11176 -0.9906) (xy -0.32512 -0.9906) (xy -0.4191 -0.50038) (xy -0.44704 -0.34798)
+      (xy -0.47752 -0.20828) (xy -0.50038 -0.09144) (xy -0.51816 -0.00762) (xy -0.52832 0.03556)
+      (xy -0.52832 0.0381) (xy -0.53848 0.03048) (xy -0.55372 -0.02032) (xy -0.57658 -0.1143)
+      (xy -0.60706 -0.2413) (xy -0.64008 -0.40132) (xy -0.6477 -0.4445) (xy -0.75184 -0.9779)
+      (xy -0.96012 -0.98552) (xy -1.1684 -0.99314) (xy -1.1684 0) (xy -1.1684 0.9906)
+      (xy -1.0287 0.9906) (xy -0.889 0.9906) (xy -0.88646 0.31242) (xy -0.88646 -0.3683)
+      (xy -0.81534 0) (xy -0.78232 0.16764) (xy -0.7493 0.35052) (xy -0.71628 0.52832)
+      (xy -0.68834 0.67818) (xy -0.6858 0.68072) (xy -0.62992 0.99314) (xy -0.53848 0.98552)
+      (xy -0.44704 0.9779) (xy -0.32004 0.2794) (xy -0.1905 -0.4191) (xy -0.18542 0.28702)
+      (xy -0.1778 0.9906) (xy -0.0381 0.9906) (xy 0.1016 0.9906) (xy 0.1016 2.02946)
+      (xy -0.05588 2.032) (xy -0.80772 2.032) (xy -1.35128 1.58496) (xy -1.49352 1.46558)
+      (xy -1.62306 1.3589) (xy -1.73482 1.26492) (xy -1.82372 1.19126) (xy -1.88722 1.14046)
+      (xy -1.91262 1.1176) (xy -1.91516 1.1176) (xy -1.92278 1.08712) (xy -1.94056 1.016)
+      (xy -1.96342 0.90678) (xy -1.9939 0.76708) (xy -2.02438 0.59944) (xy -2.05994 0.41656)
+      (xy -2.06756 0.3683) (xy -2.20218 -0.36322) (xy -1.83896 -1.00076) (xy -1.74498 -1.16332)
+      (xy -1.65862 -1.31318) (xy -1.57988 -1.44272) (xy -1.51638 -1.54432) (xy -1.47066 -1.61798)
+      (xy -1.44526 -1.651) (xy -1.44272 -1.65354) (xy -1.41224 -1.66624) (xy -1.33858 -1.69418)
+      (xy -1.2319 -1.73482) (xy -1.09474 -1.78816) (xy -0.93726 -1.84658) (xy -0.76454 -1.91008)
+      (xy -0.74422 -1.9177) (xy -0.0762 -2.16408) (xy 0.61976 -1.91516) (xy 1.31572 -1.6637)
+      (xy 1.68148 -1.04394) (xy 1.77546 -0.88392) (xy 1.86182 -0.7366) (xy 1.93548 -0.60706)
+      (xy 1.9939 -0.50546) (xy 2.03454 -0.43434) (xy 2.05232 -0.40132) (xy 2.05486 -0.40132)
+      (xy 2.05486 -0.40132)) (layer F.SilkS) (width 0.00254))
+    (fp_poly (pts (xy 0.8636 -0.37338) (xy 0.86106 -0.2413) (xy 0.8509 -0.14986) (xy 0.8255 -0.09144)
+      (xy 0.7874 -0.0635) (xy 0.72898 -0.0508) (xy 0.70612 -0.0508) (xy 0.65786 -0.05842)
+      (xy 0.62992 -0.09144) (xy 0.6096 -0.14478) (xy 0.59182 -0.26416) (xy 0.58674 -0.39878)
+      (xy 0.59944 -0.52832) (xy 0.61722 -0.6096) (xy 0.6604 -0.68072) (xy 0.72136 -0.70866)
+      (xy 0.78994 -0.69088) (xy 0.81534 -0.67056) (xy 0.8382 -0.64516) (xy 0.8509 -0.60452)
+      (xy 0.85852 -0.54102) (xy 0.8636 -0.44704) (xy 0.8636 -0.37338) (xy 0.8636 -0.37338)) (layer F.SilkS) (width 0.00254))
+  )
   (gr_line (start 159.55 87.67) (end 140.45 87.67) (angle 90) (layer Edge.Cuts) (width 0.2))

Commit message: ICSP keepout recognized on MW. Silks, gerbers.
Parts:
- moved PrettyLady 0.32 mm to (150.4, 106.6)
Other:
- board text added: "Design by Robert Powers"
- board text added: "Licensed TAPR OHL tapr.org/OHL"
- board text added: "© M9Design.co 2013"
- board text removed: "MeshThing v2.0 © M9Design.co 2013 Designed by Robert Powers"
- board text removed: "OpenHardware Under TAPR OHL tapr.org/OHL"
Changed lines of the file:
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@@
     (links 85)
     (no_connects 0)
-    (area 136.629829 85.2768 169.635341 113.0282)
+    (area 140.349999 87.569999 159.650001 112.430001)
     (thickness 1.6)
-    (drawings 7)
+    (drawings 8)
     (tracks 588)
     (zones 0)
@@
   )
   (layers
-    (15 F.Cu signal)
+    (15 F.Cu signal hide)
     (2 Inner2.Cu power hide)
     (1 Inner1.Cu signal hide)
@@
     (19 F.Paste user hide)
     (20 B.SilkS user)
-    (21 F.SilkS user)
+    (21 F.SilkS user hide)
     (22 B.Mask user)
     (23 F.Mask user)
@@
     (mod_text_size 1.5 1.5)
     (mod_text_width 0.15)
-    (pad_size 1 0.7)
-    (pad_drill 0.6299)
+    (pad_size 0.5 3.94)
+    (pad_drill 0)
     (pad_to_mask_clearance 0.2)
     (pad_to_paste_clearance_ratio -0.1)
     (aux_axis_origin 150 100)
     (grid_origin 150 100)
-    (visible_elements FFFFCE7B)
+    (visible_elements FFFFCE5B)
     (pcbplotparams
       (layerselection 284983303)
@@
   )
   (module _MT_MC_Pretty:_MC_LOGO-PrettyLady (layer B.Cu)
-    (at 150.27 106.86)
+    (at 150.37 106.56)
     (fp_text reference PrettyLady (at 0 -3.302) (layer B.SilkS) hide
       (effects (font (thickness 0.3048)) (justify mirror))
@@
       (net 37 PF7))
   )
-  (module _MT_MC_Pretty:_MT_IFA-2.4GHzPCBAntenna (layer F.Cu)
-    (at 150 90.595)
-    (fp_text reference A1 (at 0 -3.84) (layer F.SilkS) hide
-      (effects (font (size 1.5 1.5) (thickness 0.15)))
-    )
-    (fp_text value ANTENNA (at 0 4.32) (layer F.SilkS) hide
-      (effects (font (size 1.5 1.5) (thickness 0.15)))
-    )
-    (fp_text user "Comment Line - Ground plane fill 2nd layer below middle of line." (at 1.84 5.64) (layer F.SilkS) hide
-      (effects (font (size 0.5 0.5) (thickness 0.125)))
-    )
-    (fp_text user CuKeepout (at 7.89 -3.48) (layer F.SilkS) hide
-      (effects (font (size 1 1) (thickness 0.15)))
-    )
-    (fp_text user ViaToGnd (at -6.63 3.33) (layer F.SilkS) hide
-      (effects (font (size 0.5 0.5) (thickness 0.125)))
-    )
-    (fp_line (start -6.85 2.4) (end -6.45 2.4) (layer Cmts.User) (width 0.15))
-    (fp_line (start -6.65 2.6) (end -6.65 2.2) (layer Cmts.User) (width 0.15))
-    (fp_line (start -7.6 2.35) (end 7.6 2.35) (layer Cmts.User) (width 0.1))
-    (fp_text user "FeedPoint-50 Ohm" (at -0.57 2.42) (layer F.SilkS) hide
-      (effects (font (size 0.5 0.5) (thickness 0.125)))
-    )
-    (fp_line (start 7.6 -2.85) (end -7.6 -2.85) (layer Eco1.User) (width 0.15))
-    (fp_line (start 7.6 2.85) (end 7.6 -2.85) (layer Eco1.User) (width 0.15))
-    (fp_line (start -7.6 2.85) (end 7.6 2.85) (layer Eco1.User) (width 0.15))
-    (fp_line (start -7.6 2.85) (end -7.6 -2.85) (layer Eco1.User) (width 0.15))
-    (pad "" smd rect (at 0.15 -0.73) (size 0.5 2.64) (layers F.Cu F.Mask))
-    (pad "" smd rect (at 2.35 -0.73) (size 0.5 2.64) (layers F.Cu F.Mask))
-    (pad "" smd rect (at 4.85 -0.73) (size 0.5 2.64) (layers F.Cu F.Mask))
-    (pad "" smd rect (at -2.35 -0.73) (size 0.5 2.64) (layers F.Cu F.Mask))
-    (pad "" smd rect (at 1.25 -2.3) (size 2.7 0.5) (layers F.Cu F.Mask))
-    (pad "" smd rect (at 5.95 -2.3) (size 2.7 0.5) (layers F.Cu F.Mask))
-    (pad "" smd rect (at 3.6 0.34) (size 2 0.5) (layers F.Cu F.Mask))
-    (pad "" smd rect (at -1.1 0.34) (size 2 0.5) (layers F.Cu F.Mask))
-    (pad "" smd rect (at 7.05 -0.08) (size 0.5 3.94) (layers F.Cu F.Mask))
-    (pad "" smd rect (at -4.6 -2.3) (size 5 0.5) (layers F.Cu F.Mask))
-    (pad 1 smd rect (at -4.55 0.4) (size 0.5 4.9) (layers F.Cu F.Mask)
-      (net 5 "Net-(A1-Pad1)"))
-    (pad 2 smd rect (at -6.65 0.4) (size 0.9 4.9) (layers F.Cu F.Mask)
-      (net 2 GND))
-  )
   (module _MT_M9Logo-Scaled:M9Logo-scaled (layer F.Cu)
     (at 143 90.55)
@@
       (xy 0.85852 -0.54102) (xy 0.8636 -0.44704) (xy 0.8636 -0.37338) (xy 0.8636 -0.37338)) (layer F.SilkS) (width 0.00254))
   )
+  (module _MT_MC_Pretty:_MT_IFA-2.4GHzPCBAntenna (layer F.Cu)
+    (at 150 90.595)
+    (fp_text reference A1 (at 0 -3.84) (layer F.SilkS) hide
+      (effects (font (size 1.5 1.5) (thickness 0.15)))
+    )
+    (fp_text value ANTENNA (at 0 4.32) (layer F.SilkS) hide
+      (effects (font (size 1.5 1.5) (thickness 0.15)))
+    )
+    (fp_text user "Comment Line - Ground plane fill 2nd layer below middle of line." (at 1.84 5.64) (layer F.SilkS) hide
+      (effects (font (size 0.5 0.5) (thickness 0.125)))
+    )
+    (fp_text user CuKeepout (at 7.89 -3.48) (layer F.SilkS) hide
+      (effects (font (size 1 1) (thickness 0.15)))
+    )
+    (fp_text user ViaToGnd (at -6.63 3.33) (layer F.SilkS) hide
+      (effects (font (size 0.5 0.5) (thickness 0.125)))
+    )
+    (fp_line (start -6.85 2.4) (end -6.45 2.4) (layer Cmts.User) (width 0.15))
+    (fp_line (start -6.65 2.6) (end -6.65 2.2) (layer Cmts.User) (width 0.15))
+    (fp_line (start -7.6 2.35) (end 7.6 2.35) (layer Cmts.User) (width 0.1))
+    (fp_text user "FeedPoint-50 Ohm" (at -0.57 2.42) (layer F.SilkS) hide
+      (effects (font (size 0.5 0.5) (thickness 0.125)))
+    )
+    (fp_line (start 7.6 -2.85) (end -7.6 -2.85) (layer Eco1.User) (width 0.15))
+    (fp_line (start 7.6 2.85) (end 7.6 -2.85) (layer Eco1.User) (width 0.15))
+    (fp_line (start -7.6 2.85) (end 7.6 2.85) (layer Eco1.User) (width 0.15))
+    (fp_line (start -7.6 2.85) (end -7.6 -2.85) (layer Eco1.User) (width 0.15))
+    (pad "" smd rect (at 0.15 -0.73) (size 0.5 2.64) (layers F.Cu))
+    (pad "" smd rect (at 2.35 -0.73) (size 0.5 2.64) (layers F.Cu))
+    (pad "" smd rect (at 4.85 -0.73) (size 0.5 2.64) (layers F.Cu))
+    (pad "" smd rect (at -2.35 -0.73) (size 0.5 2.64) (layers F.Cu))
+    (pad "" smd rect (at 1.25 -2.3) (size 2.7 0.5) (layers F.Cu))
+    (pad "" smd rect (at 5.95 -2.3) (size 2.7 0.5) (layers F.Cu))
+    (pad "" smd rect (at 3.6 0.34) (size 2 0.5) (layers F.Cu))
+    (pad "" smd rect (at -1.1 0.34) (size 2 0.5) (layers F.Cu))
+    (pad "" smd rect (at 7.05 -0.08) (size 0.5 3.94) (layers F.Cu))
+    (pad "" smd rect (at -4.6 -2.3) (size 5 0.5) (layers F.Cu))
+    (pad 1 smd rect (at -4.55 0.4) (size 0.5 4.9) (layers F.Cu)
+      (net 5 "Net-(A1-Pad1)"))
+    (pad 2 smd rect (at -6.65 0.4) (size 0.9 4.9) (layers F.Cu)
+      (net 2 GND))
+  )
+  (gr_text "Design    by \nRobert Powers" (at 158.2 97.81) (layer B.SilkS)
+    (effects (font (size 1 1) (thickness 0.25)) (justify left mirror))
+  )
   (gr_line (start 159.55 87.67) (end 140.45 87.67) (angle 90) (layer Edge.Cuts) (width 0.2))
   (gr_line (start 159.55 112.33) (end 159.55 87.67) (angle 90) (layer Edge.Cuts) (width 0.2))
   (gr_line (start 140.45 112.33) (end 159.55 112.33) (angle 90) (layer Edge.Cuts) (width 0.2))
   (gr_line (start 140.45 87.7) (end 140.45 112.31) (angle 90) (layer Edge.Cuts) (width 0.2))
-  (gr_text "OpenHardware\nUnder \nTAPR OHL\ntapr.org/OHL" (at 158.19 103.14) (layer B.SilkS)
+  (gr_text "      Licensed\nTAPR OHL\ntapr.org/OHL" (at 158.2 103.48) (layer B.SilkS)
     (effects (font (size 0.8 0.8) (thickness 0.2)) (justify left mirror))
   )
@@
     (effects (font (size 0.9 0.9) (thickness 0.225)))
   )
-  (gr_text "MeshThing v2.0\n© M9Design.co 2013\nDesigned by \nRobert Powers\n" (at 158.19 97.16) (layer B.SilkS)
+  (gr_text "© M9Design.co 2013\n" (at 158.25 94.65) (layer B.SilkS)
     (effects (font (size 1 1) (thickness 0.25)) (justify left mirror))
   )
